File: micropad8x8/micropad8x8.kicad_pcb (KiCad board)
At the start: 2 copper layers, 32 parts

Commit message: updated pcb
Parts:
- added U1: Raspberry_Pi_Pico, MCU:Raspberry_Pi_Pico, F.Cu at (186.4, 64.0)
- S1, S10, S11, S12, S13, S14, S15, S16, S2, S3, S4, S5, S6, S7, S8, S9: footprint Button_Switch_Keyboard:SW_Cherry_MX_1.00u_PCB -> MX:MX_PCB_1.00u

Commit message: update pcb
Parts:
- added REF**: MountingHole_3.2mm_M3_Pad_TopBottom, MountingHole:MountingHole_3.2mm_M3_Pad_TopBottom, F.Cu at (276.4, 101.1)
- added REF**: MountingHole_3.2mm_M3_Pad_TopBottom, MountingHole:MountingHole_3.2mm_M3_Pad_TopBottom, F.Cu at (276.4, 20.1)
- added REF**: MountingHole_3.2mm_M3_Pad_TopBottom, MountingHole:MountingHole_3.2mm_M3_Pad_TopBottom, F.Cu at (140.7, 101.6)
- added REF**: MountingHole_3.2mm_M3_Pad_TopBottom, MountingHole:MountingHole_3.2mm_M3_Pad_TopBottom, F.Cu at (26.4, 101.6)
- added REF**: MountingHole_3.2mm_M3_Pad_TopBottom, MountingHole:MountingHole_3.2mm_M3_Pad_TopBottom, F.Cu at (140.7, 20.6)
- added REF**: MountingHole_3.2mm_M3_Pad_TopBottom, MountingHole:MountingHole_3.2mm_M3_Pad_TopBottom, F.Cu at (162.1, 20.1)
- added REF**: MountingHole_3.2mm_M3_Pad_TopBottom, MountingHole:MountingHole_3.2mm_M3_Pad_TopBottom, F.Cu at (162.1, 101.1)
- added REF**: MountingHole_3.2mm_M3_Pad_TopBottom, MountingHole:MountingHole_3.2mm_M3_Pad_TopBottom, F.Cu at (26.4, 20.6)
- D1, D10, D11, D12, D13, D14, D15, D16, D2, D3, D4, D5, D6, D7, D8, D9: moved to B.Cu
- moved S13 109.1 mm to (38.3, 89.7)
- moved D13 97.8 mm to (47.8, 92.5), turned to 90 degrees
- moved D9 97.3 mm to (47.8, 73.5), turned to 90 degrees
- moved D5 97.0 mm to (47.8, 54.4), turned to 90 degrees
- moved D1 97.0 mm to (47.8, 35.4), turned to 90 degrees
- moved S14 83.5 mm to (57.3, 89.7)
- moved S9 82.9 mm to (38.3, 70.6)
- moved D14 78.5 mm to (66.8, 92.5), turned to 90 degrees
- moved D2 78.1 mm to (66.8, 35.4), turned to 90 degrees
- moved D10 78.1 mm to (66.8, 73.5), turned to 90 degrees
- moved D6 77.9 mm to (66.8, 54.4), turned to 90 degrees
- moved S4 71.5 mm to (95.4, 32.5)
- moved U1 61.2 mm to (127.0, 49.0)
- moved S15 59.9 mm to (76.4, 89.7)
- moved D3 59.6 mm to (85.9, 35.4), turned to 90 degrees
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Connections:
- S12 pad 1: Col 2 -> Col 3
- S16 pad 1: Col 2 -> Col 3
- S4 pad 1: Col 2 -> Col 3
- S8 pad 1: Col 2 -> Col 3
- U1 pad 7: Col 2 -> Col 3
Routing:
- net Col 0: track 0.00 -> 148.6 mm
- net Col 1: track 0.00 -> 130.3 mm
- net Col 2: track 0.00 -> 111.9 mm
- net Col 3: track 0.00 -> 94.6 mm
- net Row 3: track 0.00 -> 93.1 mm
- net Row 0: track 0.00 -> 87.7 mm
- net Row 2: track 0.00 -> 79.1 mm
- net Row 1: track 0.00 -> 73.9 mm
- net Net-(D8-A): track 0.00 -> 7.12 mm
- net Net-(D7-A): track 0.00 -> 7.12 mm
- net Net-(D6-A): track 0.00 -> 7.12 mm
- net Net-(D5-A): track 0.00 -> 7.12 mm
- net Net-(D4-A): track 0.00 -> 7.12 mm
- net Net-(D3-A): track 0.00 -> 7.12 mm
- net Net-(D2-A): track 0.00 -> 7.12 mm
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- added copper zone on B.Cu, net (none)
- added copper zone on F.Cu, net (none)
Other:
- board outline added: 257.2 x 88.6 mm
