File: micropad8x8/micropad8x8.kicad_sch (KiCad schematic)
At the start: 33 parts, among them U1 Raspberry_Pi_Pico

Commit message: updated pcb
Parts:
- S1, S10, S11, S12, S13, S14, S15, S16, S2, S3, S4, S5, S6, S7, S8, S9: footprint Button_Switch_Keyboard:SW_Cherry_MX_1.00u_PCB -> MX:MX_PCB_1.00u
- U1: footprint Extra_MCU:Raspberry_Pi_Pico -> MCU:Raspberry_Pi_Pico
Changed lines of the file:
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@@
       (effects (font (size 1.27 1.27)))
     )
-    (property "Footprint" "Button_Switch_Keyboard:SW_Cherry_MX_1.00u_PCB" (at 189.23 66.04 0)
+    (property "Footprint" "MX:MX_PCB_1.00u" (at 189.23 66.04 0)
       (effects (font (size 1.27 1.27)) hide)
     )
@@
       (effects (font (size 1.27 1.27)))
     )
-    (property "Footprint" "Button_Switch_Keyboard:SW_Cherry_MX_1.00u_PCB" (at 176.53 123.19 0)
+    (property "Footprint" "MX:MX_PCB_1.00u" (at 176.53 123.19 0)
       (effects (font (size 1.27 1.27)) hide)
     )
@@
       (effects (font (size 1.27 1.27)))
     )
-    (property "Footprint" "Button_Switch_Keyboard:SW_Cherry_MX_1.00u_PCB" (at 189.23 123.19 0)
+    (property "Footprint" "MX:MX_PCB_1.00u" (at 189.23 123.19 0)
       (effects (font (size 1.27 1.27)) hide)
     )
@@
       (effects (font (size 1.27 1.27)))
     )
-    (property "Footprint" "Button_Switch_Keyboard:SW_Cherry_MX_1.00u_PCB" (at 163.83 85.09 0)
+    (property "Footprint" "MX:MX_PCB_1.00u" (at 163.83 85.09 0)
       (effects (font (size 1.27 1.27)) hide)
     )
@@
       (effects (font (size 1.27 1.27)))
     )
-    (property "Footprint" "Button_Switch_Keyboard:SW_Cherry_MX_1.00u_PCB" (at 201.93 66.04 0)
+    (property "Footprint" "MX:MX_PCB_1.00u" (at 201.93 66.04 0)
       (effects (font (size 1.27 1.27)) hide)
     )
@@
       (effects (font (size 1.27 1.27)))
     )
-    (property "Footprint" "Button_Switch_Keyboard:SW_Cherry_MX_1.00u_PCB" (at 163.83 66.04 0)
+    (property "Footprint" "MX:MX_PCB_1.00u" (at 163.83 66.04 0)
       (effects (font (size 1.27 1.27)) hide)
     )
@@
       (effects (font (size 1.27 1.27)))
     )
-    (property "Footprint" "Button_Switch_Keyboard:SW_Cherry_MX_1.00u_PCB" (at 201.93 123.19 0)
+    (property "Footprint" "MX:MX_PCB_1.00u" (at 201.93 123.19 0)
       (effects (font (size 1.27 1.27)) hide)
     )
@@
       (effects (font (size 1.27 1.27)))
     )
-    (property "Footprint" "Button_Switch_Keyboard:SW_Cherry_MX_1.00u_PCB" (at 201.93 85.09 0)
+    (property "Footprint" "MX:MX_PCB_1.00u" (at 201.93 85.09 0)
       (effects (font (size 1.27 1.27)) hide)
     )
@@
       (effects (font (size 1.27 1.27)))
     )
-    (property "Footprint" "Button_Switch_Keyboard:SW_Cherry_MX_1.00u_PCB" (at 189.23 104.14 0)
+    (property "Footprint" "MX:MX_PCB_1.00u" (at 189.23 104.14 0)
       (effects (font (size 1.27 1.27)) hide)
     )
@@
       (effects (font (size 1.27 1.27)))
     )
-    (property "Footprint" "Button_Switch_Keyboard:SW_Cherry_MX_1.00u_PCB" (at 176.53 104.14 0)
+    (property "Footprint" "MX:MX_PCB_1.00u" (at 176.53 104.14 0)
       (effects (font (size 1.27 1.27)) hide)
     )
@@
       (effects (font (size 1.27 1.27)))
     )
-    (property "Footprint" "Button_Switch_Keyboard:SW_Cherry_MX_1.00u_PCB" (at 176.53 66.04 0)
+    (property "Footprint" "MX:MX_PCB_1.00u" (at 176.53 66.04 0)
       (effects (font (size 1.27 1.27)) hide)
     )
@@
       (effects (font (size 1.27 1.27)))
     )
-    (property "Footprint" "Button_Switch_Keyboard:SW_Cherry_MX_1.00u_PCB" (at 176.53 85.09 0)
+    (property "Footprint" "MX:MX_PCB_1.00u" (at 176.53 85.09 0)
       (effects (font (size 1.27 1.27)) hide)
     )
@@
       (effects (font (size 1.27 1.27)))
     )
-    (property "Footprint" "Button_Switch_Keyboard:SW_Cherry_MX_1.00u_PCB" (at 163.83 104.14 0)
+    (property "Footprint" "MX:MX_PCB_1.00u" (at 163.83 104.14 0)
       (effects (font (size 1.27 1.27)) hide)
     )
@@
       (effects (font (size 1.27 1.27)))
     )
-    (property "Footprint" "Extra_MCU:Raspberry_Pi_Pico" (at 102.87 62.23 0)
+    (property "Footprint" "MCU:Raspberry_Pi_Pico" (at 102.87 62.23 0)
       (effects (font (size 1.27 1.27)) hide)
     )
@@
       (effects (font (size 1.27 1.27)))
     )
-    (property "Footprint" "Button_Switch_Keyboard:SW_Cherry_MX_1.00u_PCB" (at 163.83 123.19 0)
+    (property "Footprint" "MX:MX_PCB_1.00u" (at 163.83 123.19 0)
       (effects (font (size 1.27 1.27)) hide)
     )
@@
       (effects (font (size 1.27 1.27)))
     )
-    (property "Footprint" "Button_Switch_Keyboard:SW_Cherry_MX_1.00u_PCB" (at 189.23 85.09 0)
+    (property "Footprint" "MX:MX_PCB_1.00u" (at 189.23 85.09 0)
       (effects (font (size 1.27 1.27)) hide)
     )
@@
       (effects (font (size 1.27 1.27)))
     )
-    (property "Footprint" "Button_Switch_Keyboard:SW_Cherry_MX_1.00u_PCB" (at 201.93 104.14 0)
-      (effects (font (size 1.27 1.27)) hide)
-    )
+    (property "Footprint" "MX:MX_PCB_1.00u" (at 201.93 104.14 0)
+      (effects (font (size 1.27 1.27)) hide)
+    )

Commit message: update pcb
Connections:
- net Col 2: no longer S12.1, S16.1, S4.1, S8.1, U1.7 (GPIO5)
- new net Col 3: S12.1, S16.1, S4.1, S8.1, U1.7 (GPIO5)
Changed lines of the file:
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@@
     )
   )
-  (global_label "Col 2" (shape input) (at 199.39 54.61 90) (fields_autoplaced)
+  (global_label "Col 3" (shape input) (at 199.39 54.61 90) (fields_autoplaced)
     (effects (font (size 1.27 1.27)) (justify left))
     (property "Intersheetrefs" "${INTERSHEET_REFS}" (at 199.39 46.3635 90)
@@
     )
   )
-  (global_label "Col 2" (shape input) (at 87.63 83.82 180) (fields_autoplaced)
+  (global_label "Col 3" (shape input) (at 87.63 83.82 180) (fields_autoplaced)
     (effects (font (size 1.27 1.27)) (justify right))
     (property "Intersheetrefs" "${INTERSHEET_REFS}" (at 79.3835 83.82 0)
